File: Harware Design/file57AF0630.sch (KiCad schematic (older format))
At the start: 36 parts, among them Q3 BC849, Q4 BC849, Q5 BC849, Q6 BC849, SW10 9, SW11 0, SW12 A, SW13 B, SW14 5, SW15 6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

Commit message: RGB LED and D4 footprints are changed
Parts:
- AFF1, AFF2, AFF3, AFF4: footprint (none) -> Displays_7-Segment:7SegmentLED_LTS6760_LTS6780
- JP1: footprint (none) -> Pin_Headers:Pin_Header_Straight_1x08
- Q3, Q4, Q5, Q6: footprint (none) -> TO_SOT_Packages_SMD:SOT-23
- R37, R38, R39, R40, R41, R42, R43, R44: footprint (none) -> Resistors_SMD:R_0603_HandSoldering
- RR1, RR2: footprint (none) -> Resistors_ThroughHole:Resistor_Array_SIP8
- S1: footprint (none) -> Housings_DIP:DIP-16_W7.62mm_LongPads
- SW10, SW11, SW12, SW13, SW14, SW15, SW16, SW17, SW18, SW19, SW20, SW21, SW6, SW7, SW8, SW9: footprint (none) -> EE:SW_PUSH_SMALL_2pin_3D_xl_v1
Changed lines of the file:
@@
 EESchema Schematic File Version 2
+LIBS:One Base Board-rescue
 LIBS:power
 LIBS:device
@@
 LIBS:contrib
 LIBS:valves
-LIBS:MCU_BaseBoard-cache
-LIBS:file549BE66B-cache
-LIBS:usb to serial-cache
-LIBS:TXB0104 Level translator-cache
-LIBS:ExploreM3
 LIBS:One Base Board-cache
 EELAYER 25 0
@@
 F 0 "SW9" H 1250 6075 70  0000 C CNN
 F 1 "F" H 1250 5875 70  0000 C CNN
-F 2 "" H 1250 5975 60  0001 C CNN
+F 2 "EE:SW_PUSH_SMALL_2pin_3D_xl_v1" H 1250 5975 60  0001 C CNN
 F 3 "" H 1250 5975 60  0001 C CNN
 	1    1250 5975
@@
 F 0 "SW8" H 1250 5525 70  0000 C CNN
 F 1 "E" H 1250 5325 70  0000 C CNN
-F 2 "" H 1250 5425 60  0001 C CNN
+F 2 "EE:SW_PUSH_SMALL_2pin_3D_xl_v1" H 1250 5425 60  0001 C CNN
 F 3 "" H 1250 5425 60  0001 C CNN
 	1    1250 5425
@@
 F 0 "SW6" H 1250 4425 70  0000 C CNN
 F 1 "C" H 1250 4225 70  0000 C CNN
-F 2 "" H 1250 4325 60  0001 C CNN
+F 2 "EE:SW_PUSH_SMALL_2pin_3D_xl_v1" H 1250 4325 60  0001 C CNN
 F 3 "" H 1250 4325 60  0001 C CNN
 	1    1250 4325
@@
 F 0 "SW13" H 2550 6075 70  0000 C CNN
 F 1 "B" H 2550 5875 70  0000 C CNN
-F 2 "" H 2550 5975 60  0001 C CNN
+F 2 "EE:SW_PUSH_SMALL_2pin_3D_xl_v1" H 2550 5975 60  0001 C CNN
 F 3 "" H 2550 5975 60  0001 C CNN
 	1    2550 5975
@@
 F 0 "SW12" H 2550 5525 70  0000 C CNN
 F 1 "A" H 2550 5325 70  0000 C CNN
-F 2 "" H 2550 5425 60  0001 C CNN
+F 2 "EE:SW_PUSH_SMALL_2pin_3D_xl_v1" H 2550 5425 60  0001 C CNN
 F 3 "" H 2550 5425 60  0001 C CNN
 	1    2550 5425
@@
 F 0 "SW11" H 2550 4975 70  0000 C CNN
 F 1 "0" H 2550 4775 70  0000 C CNN
-F 2 "" H 2550 4875 60  0001 C CNN
+F 2 "EE:SW_PUSH_SMALL_2pin_3D_xl_v1" H 2550 4875 60  0001 C CNN
 F 3 "" H 2550 4875 60  0001 C CNN
 	1    2550 4875
@@
 F 0 "SW10" H 2550 4425 70  0000 C CNN
 F 1 "9" H 2550 4225 70  0000 C CNN
-F 2 "" H 2550 4325 60  0001 C CNN
+F 2 "EE:SW_PUSH_SMALL_2pin_3D_xl_v1" H 2550 4325 60  0001 C CNN
 F 3 "" H 2550 4325 60  0001 C CNN
 	1    2550 4325
@@
 F 0 "SW17" H 3750 6075 70  0000 C CNN
 F 1 "8" H 3750 5875 70  0000 C CNN
-F 2 "" H 3750 5975 60  0001 C CNN
+F 2 "EE:SW_PUSH_SMALL_2pin_3D_xl_v1" H 3750 5975 60  0001 C CNN
 F 3 "" H 3750 5975 60  0001 C CNN
 	1    3750 5975
@@
 F 0 "SW16" H 3750 5525 70  0000 C CNN
 F 1 "7" H 3750 5325 70  0000 C CNN
-F 2 "" H 3750 5425 60  0001 C CNN
+F 2 "EE:SW_PUSH_SMALL_2pin_3D_xl_v1" H 3750 5425 60  0001 C CNN
 F 3 "" H 3750 5425 60  0001 C CNN
 	1    3750 5425
@@
 F 0 "SW15" H 3750 4975 70  0000 C CNN
 F 1 "6" H 3750 4775 70  0000 C CNN
-F 2 "" H 3750 4875 60  0001 C CNN
+F 2 "EE:SW_PUSH_SMALL_2pin_3D_xl_v1" H 3750 4875 60  0001 C CNN
 F 3 "" H 3750 4875 60  0001 C CNN
 	1    3750 4875
@@
 F 0 "SW14" H 3750 4425 70  0000 C CNN
 F 1 "5" H 3750 4225 70  0000 C CNN
-F 2 "" H 3750 4325 60  0001 C CNN
+F 2 "EE:SW_PUSH_SMALL_2pin_3D_xl_v1" H 3750 4325 60  0001 C CNN
 F 3 "" H 3750 4325 60  0001 C CNN
 	1    3750 4325
@@
 F 0 "SW21" H 4950 6075 70  0000 C CNN
 F 1 "4" H 4950 5875 70  0000 C CNN
-F 2 "" H 4950 5975 60  0001 C CNN
+F 2 "EE:SW_PUSH_SMALL_2pin_3D_xl_v1" H 4950 5975 60  0001 C CNN
 F 3 "" H 4950 5975 60  0001 C CNN
 	1    4950 5975
@@
 F 0 "SW20" H 4950 5525 70  0000 C CNN
 F 1 "3" H 4950 5325 70  0000 C CNN
-F 2 "" H 4950 5425 60  0001 C CNN
+F 2 "EE:SW_PUSH_SMALL_2pin_3D_xl_v1" H 4950 5425 60  0001 C CNN
 F 3 "" H 4950 5425 60  0001 C CNN
 	1    4950 5425
@@
 F 0 "SW19" H 4950 4975 70  0000 C CNN
 F 1 "2" H 4950 4775 70  0000 C CNN
-F 2 "" H 4950 4875 60  0001 C CNN
+F 2 "EE:SW_PUSH_SMALL_2pin_3D_xl_v1" H 4950 4875 60  0001 C CNN
 F 3 "" H 4950 4875 60  0001 C CNN
 	1    4950 4875
@@
 F 0 "SW18" H 4950 4425 70  0000 C CNN
 F 1 "1" H 4950 4225 70  0000 C CNN
-F 2 "" H 4950 4325 60  0001 C CNN
+F 2 "EE:SW_PUSH_SMALL_2pin_3D_xl_v1" H 4950 4325 60  0001 C CNN
 F 3 "" H 4950 4325 60  0001 C CNN
 	1    4950 4325
@@
 F 0 "SW7" H 1250 4975 70  0000 C CNN
 F 1 "D" H 1250 4775 70  0000 C CNN
-F 2 "" H 1250 4875 60  0001 C CNN
+F 2 "EE:SW_PUSH_SMALL_2pin_3D_xl_v1" H 1250 4875 60  0001 C CNN
 F 3 "" H 1250 4875 60  0001 C CNN
 	1    1250 4875
@@
 F 0 "RR1" H 6500 5025 50  0000 C CNN
 F 1 "RR8" V 6480 4475 50  0000 C CNN
-F 2 "" H 6450 4475 60  0001 C CNN
+F 2 "Resistors_ThroughHole:Resistor_Array_SIP8" H 6450 4475 60  0001 C CNN
 F 3 "" H 6450 4475 60  0000 C CNN
 	1    6450 4475
@@
 F 0 "S1" H 9400 5200 50  0000 L BNN
 F 1 "SW_DIP-8" H 9400 4175 50  0000 L BNN
-F 2 "" H 9600 4925 50  0001 C CNN
+F 2 "Housings_DIP:DIP-16_W7.62mm_LongPads" H 9600 4925 50  0001 C CNN
 F 3 "" H 9600 4775 60  0001 C CNN
 	1    9600 4775
@@
 F 0 "JP1" H 8350 5305 50  0000 L BNN
 F 1 "SWITCH_ARRAY" H 8350 4275 50  0000 L BNN
-F 2 "" H 8550 4925 50  0001 C CNN
+F 2 "Pin_Headers:Pin_Header_Straight_1x08" H 8550 4925 50  0001 C CNN
 F 3 "" H 8550 4775 60  0001 C CNN
 	1    8550 4775
@@
 F 0 "RR2" H 9200 5275 70  0000 C CNN
 F 1 "RR8" V 9180 4725 70  0000 C CNN
-F 2 "" H 9150 4725 60  0001 C CNN
+F 2 "Resistors_ThroughHole:Resistor_Array_SIP8" H 9150 4725 60  0001 C CNN
 F 3 "" H 9150 4725 60  0001 C CNN
 	1    9150 4725
@@
 F 0 "R44" V 9305 2150 50  0000 C CNN
 F 1 "1K" V 9225 2150 50  0000 C CNN
-F 2 "" H 9225 2150 60  0001 C CNN
+F 2 "Resistors_SMD:R_0603_HandSoldering" H 9225 2150 60  0001 C CNN
 F 3 "" H 9225 2150 60  0001 C CNN
 	1    9225 2150
@@
 F 0 "R42" V 7805 2150 50  0000 C CNN
 F 1 "1K" V 7725 2150 50  0000 C CNN
-F 2 "" H 7725 2150 60  0001 C CNN
+F 2 "Resistors_SMD:R_0603_HandSoldering" H 7725 2150 60  0001 C CNN
 F 3 "" H 7725 2150 60  0001 C CNN
 	1    7725 2150
@@
 F 0 "R40" V 6305 2150 50  0000 C CNN
 F 1 "1K" V 6225 2150 50  0000 C CNN
-F 2 "" H 6225 2150 60  0001 C CNN
+F 2 "Resistors_SMD:R_0603_HandSoldering" H 6225 2150 60  0001 C CNN
 F 3 "" H 6225 2150 60  0001 C CNN
 	1    6225 2150
@@
 F 0 "R38" V 4805 2150 50  0000 C CNN
 F 1 "1K" V 4725 2150 50  0000 C CNN
-F 2 "" H 4725 2150 60  0001 C CNN
+F 2 "Resistors_SMD:R_0603_HandSoldering" H 4725 2150 60  0001 C CNN
 F 3 "" H 4725 2150 60  0001 C CNN
 	1    4725 2150
@@
 F 0 "AFF1" H 3675 1800 60  0000 C CNN
 F 1 "LTS-6960HR" H 3675 800 60  0000 C CNN
-F 2 "" H 3675 1250 60  0000 C CNN
+F 2 "Displays_7-Segment:7SegmentLED_LTS6760_LTS6780" H 3675 1250 60  0001 C CNN
 F 3 "~" H 3675 1250 60  0000 C CNN
 	1    3675 1250
@@
 F 0 "AFF2" H 5175 1800 60  0000 C CNN
 F 1 "LTS-6960HR" H 5175 800 60  0000 C CNN
-F 2 "" H 5175 1250 60  0000 C CNN
+F 2 "Displays_7-Segment:7SegmentLED_LTS6760_LTS6780" H 5175 1250 60  0001 C CNN
 F 3 "~" H 5175 1250 60  0000 C CNN
 	1    5175 1250
@@
 F 0 "AFF3" H 6675 1800 60  0000 C CNN
 F 1 "LTS-6960HR" H 6675 800 60  0000 C CNN
-F 2 "" H 6675 1250 60  0000 C CNN
+F 2 "Displays_7-Segment:7SegmentLED_LTS6760_LTS6780" H 6675 1250 60  0001 C CNN
 F 3 "~" H 6675 1250 60  0000 C CNN
 	1    6675 1250
@@
 F 0 "AFF4" H 8175 1800 60  0000 C CNN
 F 1 "LTS-6960HR" H 8175 800 60  0000 C CNN
-F 2 "" H 8175 1250 60  0000 C CNN
+F 2 "Displays_7-Segment:7SegmentLED_LTS6760_LTS6780" H 8175 1250 60  0001 C CNN
 F 3 "~" H 8175 1250 60  0000 C CNN
 	1    8175 1250
@@
 79 E3 73 01 AA 0D CF 9F 3C 98 C5 F6 CF AC 04 72 85 62 D7 80 77 B1 8B CB 18 6F AC E9 6A 17 BB B8
 C2 B0 6B C0 BB D8 C5 65 8C 5D 03 DE C5 2E 2E 63 EC 1A F0 2E 76 71 19 63 D7 80 77 B1 8B CB 18 BB
-06 BC 8B 5D 5C C6 F8 FF 01 52 B3 1C 8C A4 9D 25 1B 00 00 00 00 49 45 4E 44 AE 42 60 82 83
+06 BC 8B 5D 5C C6 F8 FF 01 52 B3 1C 8C A4 9D 25 1B 00 00 00 00 49 45 4E 44 AE 42 60 82 A7
 EndData
 $EndBitmap
@@
 F 0 "R37" V 4455 2350 50  0000 C CNN
 F 1 "68" V 4375 2350 50  0000 C CNN
-F 2 "" H 4375 2350 60  0001 C CNN
+F 2 "Resistors_SMD:R_0603_HandSoldering" H 4375 2350 60  0001 C CNN
 F 3 "" H 4375 2350 60  0001 C CNN
 	1    4375 2350
@@
 F 0 "R39" V 5955 2350 50  0000 C CNN
 F 1 "68" V 5875 2350 50  0000 C CNN
-F 2 "" H 5875 2350 60  0001 C CNN
+F 2 "Resistors_SMD:R_0603_HandSoldering" H 5875 2350 60  0001 C CNN
 F 3 "" H 5875 2350 60  0001 C CNN
 	1    5875 2350
@@
 F 0 "R41" V 7455 2350 50  0000 C CNN
 F 1 "68" V 7375 2350 50  0000 C CNN
-F 2 "" H 7375 2350 60  0001 C CNN
+F 2 "Resistors_SMD:R_0603_HandSoldering" H 7375 2350 60  0001 C CNN
 F 3 "" H 7375 2350 60  0001 C CNN
 	1    7375 2350
@@
 F 0 "R43" V 8955 2350 50  0000 C CNN
 F 1 "68" V 8875 2350 50  0000 C CNN
-F 2 "" H 8875 2350 60  0001 C CNN
+F 2 "Resistors_SMD:R_0603_HandSoldering" H 8875 2350 60  0001 C CNN
 F 3 "" H 8875 2350 60  0001 C CNN
 	1    8875 2350
@@
 F 0 "Q3" H 4175 2001 40  0000 R CNN
 F 1 "BC849" H 4175 2300 40  0000 R CNN
-F 2 "" H 4075 2252 29  0000 C CNN
+F 2 "TO_SOT_Packages_SMD:SOT-23" H 4075 2252 29  0001 C CNN
 F 3 "" H 4175 2150 60  0000 C CNN
 	1    4175 2150
@@
 F 0 "Q4" H 5675 2001 40  0000 R CNN
 F 1 "BC849" H 5675 2300 40  0000 R CNN
-F 2 "" H 5575 2252 29  0000 C CNN
+F 2 "TO_SOT_Packages_SMD:SOT-23" H 5575 2252 29  0001 C CNN
 F 3 "" H 5675 2150 60  0000 C CNN
 	1    5675 2150
@@
 F 0 "Q5" H 7175 2001 40  0000 R CNN
 F 1 "BC849" H 7175 2300 40  0000 R CNN
-F 2 "" H 7075 2252 29  0000 C CNN
+F 2 "TO_SOT_Packages_SMD:SOT-23" H 7075 2252 29  0001 C CNN
 F 3 "" H 7175 2150 60  0000 C CNN
 	1    7175 2150
@@
 F 0 "Q6" H 8675 2001 40  0000 R CNN
 F 1 "BC849" H 8675 2300 40  0000 R CNN
-F 2 "" H 8575 2252 29  0000 C CNN
+F 2 "TO_SOT_Packages_SMD:SOT-23" H 8575 2252 29  0001 C CNN
 F 3 "" H 8675 2150 60  0000 C CNN
 	1    8675 2150
